File: connectors.kicad_sch (KiCad schematic)
At the start: 34 parts, among them J10 1755736, J12 1755736, J13 1755736, J14 Conn_02x06_Odd_Even, J15 1755736, J16 1755736, J17 Conn_02x06_Odd_Even, J18 1755736, J19 1755736, J20 Conn_02x06_Odd_Even, J21 1755736, J22 1755736, J9 12402012E212A, Q7 STL40DN3LLH5, U3 INA236BIDDFR, U4 INA236AIDDFR, U5 INA236AIDDFR, U6 INA236AIDDFR, U9 TCPP02-M18

Commit message: PCB 2025 rev2
Parts:
- removed J9: 12402012E212A, Modelec:AMPHENOL_12402012E212A, symbol Modelec:12402012E212A
- added J11: USB_C_Receptacle_USB2.0_16P, Modelec:GCT_USB4105-GF-A, symbol Connector:USB_C_Receptacle_USB2.0_16P
- C22: value 2.2u -> 2u2
- R19: value L4CL1206LR013DNR -> 62m 0.5%
- R20, R22: value L4CL1206LR013DNR -> 13m 0.5%
- R21: value L4CL1206LR013DNR -> 20m 0.5%
- R25: value L4CL1206LR007FNR -> 7m 1%
Connections:
- net GND: now also J11.A1_B12 (GND), J11.B1_A12 (GND), J11.SH1 (SHIELD), J11.SH2, J11.SH3, J11.SH4
- net at C20.2, U9.11 (CC2C): now also J11.B5 (CC2)
- net at C22.1, D4.1 (K), R25.1: now also J11.A4_B9 (VBUS), J11.B4_A9 (VBUS)
- net at C19.1, U9.13 (CC1C): now also J11.A5 (CC1)
Other:
- moved on the sheet: C22, D4
