File: power_input_selector.kicad_sch (KiCad schematic)
At the start: 35 parts, among them Q1 SUD50P06-15, Q2 SUD50P06-15, Q3 SUD50P06-15, Q4 SUD50P06-15, Q5 SUD50P06-15, Q6 SUD50P06-15, U1 LTC4417IGN, U7 INA236BIDDFR, U8 INA236BIDDFR

Commit message: PCB 2025 rev2
Parts:
- C1, C3, C5: value 0.4u -> 0u4
- R10, R7: value 37.4k -> 37k4
- R11, R8: value 78.7k -> 78k7
- R13, R14, R15: value 8.06k -> 8k06
- R23, R24: value 4m -> 4m 0.5%
- R4: value 63.4k -> 63k4
Changed lines of the file:
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@@
 	(title_block
 		(title "Power input selector")
-		(date "2025-01-25")
-		(rev "1")
+		(date "2025-01-29")
+		(rev "2")
 		(company "Modelec")
 		(comment 1 "Shuts down all inputs with EN. Returns validity status of each line with VALID")
@@
 			)
 		)
-		(property "Value" "63.4k"
+		(property "Value" "63k4"
 			(at 106.68 114.2999 0)
 			(effects
@@
 			)
 		)
-		(property "Value" "78.7k"
+		(property "Value" "78k7"
 			(at 73.66 166.3699 0)
 			(effects
@@
 			)
 		)
-		(property "Value" "37.4k"
+		(property "Value" "37k4"
 			(at 90.17 143.5099 0)
 			(effects
@@
 			)
 		)
-		(property "Value" "8.06k"
+		(property "Value" "8k06"
 			(at 246.38 46.9899 0)
 			(effects
@@
 			)
 		)
-		(property "Value" "0.4u"
+		(property "Value" "0u4"
 			(at 220.218 46.99 0)
 			(effects
@@
 			)
 		)
-		(property "Datasheet" "~"
+		(property "Datasheet" "https://search.kemet.com/download/specsheet/ESY108M035AL4AA"
 			(at 267.97 74.93 0)
 			(effects
@@
 			)
 		)
-		(property "Value" "37.4k"
+		(property "Value" "37k4"
 			(at 73.66 173.9899 0)
 			(effects
@@
 			)
 		)
-		(property "Value" "0.4u"
+		(property "Value" "0u4"
 			(at 164.338 46.99 0)
 			(effects
@@
 			)
 		)
-		(property "Value" "78.7k"
+		(property "Value" "78k7"
 			(at 90.17 135.8899 0)
 			(effects
@@
 			)
 		)
-		(property "Value" "8.06k"
+		(property "Value" "8k06"
 			(at 190.5 46.9899 0)
 			(effects
@@
 			)
 		)
-		(property "Value" "0.4u"
+		(property "Value" "0u4"
 			(at 108.458 46.99 0)
 			(effects
@@
 			)
 		)
-		(property "Value" "8.06k"
+		(property "Value" "8k06"
 			(at 134.62 46.9899 0)
 			(effects
@@
 			)
 		)
-		(property "Value" "4m"
+		(property "Value" "4m 0.5%"
 			(at 66.04 102.8699 0)
 			(effects
@@
 			)
 		)
-		(property "Datasheet" "~"
+		(property "Datasheet" "https://s.resistor.today/shop/products/epdf/PEWF2512.pdf"
 			(at 63.5 101.6 0)
 			(effects
@@
 			)
 		)
-		(property "Value" "4m"
+		(property "Value" "4m 0.5%"
 			(at 66.04 71.1199 0)
 			(effects
@@
 			)
 		)
-		(property "Datasheet" "~"
+		(property "Datasheet" "https://s.resistor.today/shop/products/epdf/PEWF2512.pdf"
 			(at 63.5 69.85 0)
 			(effects
